File: PowerSourceArbitrator.kicad_sch (KiCad schematic)
At the start: 0 parts

Commit message: Added USB ports for board 0
Parts:
- added J1, J2: Connector_USB_C_Receptacle_USB2.0, symbol USB-C-USB-2.0-cache:Connector_USB_C_Receptacle_USB2.0
Connections:
- new net GND: J1.A1 (GND), J1.A12 (GND), J1.B1 (GND), J1.B12 (GND), J2.A1 (GND), J2.A12 (GND), J2.B1 (GND), J2.B12 (GND)
- new net VBUS: J1.A4 (VBUS), J1.A9 (VBUS), J1.B4 (VBUS), J1.B9 (VBUS), J2.A4 (VBUS), J2.A9 (VBUS), J2.B4 (VBUS), J2.B9 (VBUS)
Changed lines of the file:
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@@
 	(generator_version "10.0")
 	(paper "A4")
+	(symbol
+		(lib_id "USB-C-USB-2.0-cache:Connector_USB_C_Receptacle_USB2.0")
+		(at 57.15 147.32 270)
+		(mirror x)
+		(unit 1)
+		(body_style 1)
+		(exclude_from_sim no)
+		(in_bom yes)
+		(on_board yes)
+		(in_pos_files yes)
+		(dnp no)
+		(property "Reference" "J2"
+			(at 76.2 148.5901 90)
+			(show_name no)
+			(do_not_autoplace no)
+			(effects
+				(font
+					(size 1.27 1.27)
+				)
+				(justify left)
+			)
+		)
+		(property "Value" "Connector_USB_C_Receptacle_USB2.0"
+			(at 76.2 146.0501 90)
+			(show_name no)
+			(do_not_autoplace no)
+			(effects
+				(font
+					(size 1.27 1.27)
+				)
+				(justify left)
+			)
+		)
+		(property "Footprint" ""
+			(at 57.15 143.51 0)
+			(hide yes)
+			(show_name no)
+			(do_not_autoplace no)
+			(effects
+				(font
+					(size 1.27 1.27)
+				)
+			)
+		)
+		(property "Datasheet" ""
+			(at 57.15 143.51 0)
+			(hide yes)
+			(show_name no)
+			(do_not_autoplace no)
+			(effects
+				(font
+					(size 1.27 1.27)
+				)
+			)
+		)
+		(property "Description" ""
+			(at 57.15 147.32 0)
+			(hide yes)
+			(show_name no)
+			(do_not_autoplace no)
+			(effects
+				(font
+					(size 1.27 1.27)
+				)
+			)
+		)
+		(pin "A12"
+		)
+		(pin "A4"
+		)
+		(pin "A6"
+		)
+		(pin "B1"
+		)
+		(pin "B4"
+		)
+		(pin "A9"
+		)
+		(pin "B6"
+		)
+		(pin "B7"
+		)
+		(pin "A1"
+		)
+		(pin "B9"
+		)
+		(pin "A8"
+		)
+		(pin "B5"
+		)
+		(pin "A5"
+		)
+		(pin "A7"
+		)
+		(pin "B8"
+		)
+		(pin "B12"
+		)
+		(pin "S1"
+		)
+		(instances
+			(project "PowerSourceArbitrator"
+				(path "/388bad04-b51e-490f-8e3e-05ae0f48516d"
+					(reference "J2")
+					(unit 1)
+				)
+			)
+		)
+	)
+	(symbol
+		(lib_id "USB-C-USB-2.0-cache:Connector_USB_C_Receptacle_USB2.0")
+		(at 57.15 82.55 270)
+		(unit 1)
+		(body_style 1)
+		(exclude_from_sim no)
+		(in_bom yes)
+		(on_board yes)
+		(in_pos_files yes)
+		(dnp no)
+		(fields_autoplaced yes)
+		(property "Reference" "J1"
+			(at 76.2 81.2799 90)
+			(show_name no)
+			(do_not_autoplace no)
+			(effects
+				(font
+					(size 1.27 1.27)
+				)
+				(justify left)
+			)
+		)
+		(property "Value" "Connector_USB_C_Receptacle_USB2.0"
+			(at 76.2 83.8199 90)
+			(show_name no)
+			(do_not_autoplace no)
+			(effects
+				(font
+					(size 1.27 1.27)
+				)
+				(justify left)
+			)
+		)
+		(property "Footprint" ""
+			(at 57.15 86.36 0)
+			(hide yes)
+			(show_name no)
+			(do_not_autoplace no)
+			(effects
+				(font
+					(size 1.27 1.27)
+				)
+			)
+		)
+		(property "Datasheet" ""
+			(at 57.15 86.36 0)
+			(hide yes)
+			(show_name no)
+			(do_not_autoplace no)
+			(effects
+				(font
+					(size 1.27 1.27)
+				)
+			)
+		)
+		(property "Description" ""
+			(at 57.15 82.55 0)
+			(hide yes)
+			(show_name no)
+			(do_not_autoplace no)
+			(effects
+				(font
+					(size 1.27 1.27)
+				)
+			)
+		)
+		(pin "A12"
+		)
+		(pin "A4"
+		)
+		(pin "A6"
+		)
+		(pin "B1"
+		)
+		(pin "B4"
+		)
+		(pin "A9"
+		)
+		(pin "B6"
+		)
+		(pin "B7"
+		)
+		(pin "A1"
+		)
+		(pin "B9"
+		)
+		(pin "A8"
+		)
+		(pin "B5"
+		)
+		(pin "A5"
+		)
+		(pin "A7"
+		)
+		(pin "B8"
+		)
+		(pin "B12"
+		)
+		(pin "S1"
+		)
+		(instances
+			(project "PowerSourceArbitrator"
+				(path "/388bad04-b51e-490f-8e3e-05ae0f48516d"
+					(reference "J1")
+					(unit 1)
+				)
+			)
+		)
+	)
 	(sheet_instances
 		(path "/"
